File: Hardware/BFMC/BFMC.kicad_pcb (KiCad board)
At the start: 2 copper layers, 104.7 x 137.7 mm, 94 parts, among them J1 12V, J10 HC_SR04_1, J11 HC_SR04_2, J12 HC_SR04_3, J13 HC_SR04_4, J14 FAN_FET, J15 FAN_RAS, J16 LED_LEFT, J17 LED_RIGHT, J2 5V, J3 INIT_BLDC, J4 MOTOR_BLDC, J5 MOTOR_STEERING, J6 MOTOR_CAMERA, J7 IMU_DATA, J8 IMU_3V3, J9 IMU_5V, Q1 BSN20, Q2 BSN20, Q3 BSN20, Q4 MMBT2222A, Q5 MMBT2222A, Q6 MMBT2222A, U1 NUCLEO-F401RE, U2 RASPBERRY_PI_4B_4GB

Commit message: update temporary file in stm32
Parts:
- added R11: 0/1%, Resistor_SMD:R_0603_1608Metric_Pad0.98x0.95mm_HandSolder, B.Cu at (129.1, 89.5)
- added R12: 0/1%, Resistor_SMD:R_0603_1608Metric_Pad0.98x0.95mm_HandSolder, B.Cu at (131.1, 89.5)
- renumbered 5V to LED1, 12V to LED2, BLDC to LED3, R11 to R13, R12 to R14, R13 to R15, R14 to R16, R15 to R17, R16 to R18, R17 to R19
Connections:
- U1 pad CN10_23: MOTOR_STEERING -> MOTOR_STEERING_1
- U1 pad CN10_31: unconnected-(U1B-PB3-PadCN10_31) -> MOTOR_STEERING_2
Routing:
- net MOTOR_STEERING_1: track 0.00 -> 11.7 mm
- net MOTOR_STEERING: track 13.1 -> 6.16 mm
- net MOTOR_STEERING_2: track 0.00 -> 4.34 mm
- net GND: vias 592 -> 591
