File: Hardware/BFMC/led_buzzer.kicad_sch (KiCad schematic)
At the start: 12 parts, among them J16 LED_LEFT, J17 LED_RIGHT, Q4 MMBT2222A, Q5 MMBT2222A, Q6 MMBT2222A

Commit message: update temporary file in stm32
Parts:
- renumbered R13 to R15, R14 to R16, R15 to R17, R16 to R18, R17 to R19
Changed lines of the file:
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@@
   (symbol (lib_id "Device:R_Small_US") (at 115.57 83.82 180) (unit 1)
     (in_bom yes) (on_board yes) (dnp no) (fields_autoplaced)
-    (property "Reference" "R16" (at 118.11 82.55 0)
+    (property "Reference" "R18" (at 118.11 82.55 0)
       (effects (font (size 1.27 1.27)) (justify right))
     )
@@
       (project "BFMC"
         (path "/a702f17a-d8b6-4710-aaf3-998facd86d1b/c91c3564-35bd-4eac-9426-cc808a6c8173"
-          (reference "R16") (unit 1)
+          (reference "R18") (unit 1)
         )
       )
@@
   (symbol (lib_id "Device:R_Small_US") (at 198.12 110.49 90) (unit 1)
     (in_bom yes) (on_board yes) (dnp no) (fields_autoplaced)
-    (property "Reference" "R17" (at 198.12 104.14 90)
+    (property "Reference" "R19" (at 198.12 104.14 90)
       (effects (font (size 1.27 1.27)))
     )
@@
       (project "BFMC"
         (path "/a702f17a-d8b6-4710-aaf3-998facd86d1b/c91c3564-35bd-4eac-9426-cc808a6c8173"
-          (reference "R17") (unit 1)
+          (reference "R19") (unit 1)
         )
       )
@@
   (symbol (lib_id "Device:R_Small_US") (at 105.41 73.66 90) (unit 1)
     (in_bom yes) (on_board yes) (dnp no) (fields_autoplaced)
-    (property "Reference" "R14" (at 105.41 67.31 90)
+    (property "Reference" "R16" (at 105.41 67.31 90)
       (effects (font (size 1.27 1.27)))
     )
@@
       (project "BFMC"
         (path "/a702f17a-d8b6-4710-aaf3-998facd86d1b/c91c3564-35bd-4eac-9426-cc808a6c8173"
-          (reference "R14") (unit 1)
+          (reference "R16") (unit 1)
         )
       )
@@
   (symbol (lib_id "Device:R_Small_US") (at 104.14 121.92 90) (unit 1)
     (in_bom yes) (on_board yes) (dnp no) (fields_autoplaced)
-    (property "Reference" "R13" (at 104.14 115.57 90)
+    (property "Reference" "R15" (at 104.14 115.57 90)
       (effects (font (size 1.27 1.27)))
     )
@@
       (project "BFMC"
         (path "/a702f17a-d8b6-4710-aaf3-998facd86d1b/c91c3564-35bd-4eac-9426-cc808a6c8173"
-          (reference "R13") (unit 1)
+          (reference "R15") (unit 1)
         )
       )
@@
   (symbol (lib_id "Device:R_Small_US") (at 114.3 132.08 180) (unit 1)
     (in_bom yes) (on_board yes) (dnp no) (fields_autoplaced)
-    (property "Reference" "R15" (at 116.84 130.81 0)
+    (property "Reference" "R17" (at 116.84 130.81 0)
       (effects (font (size 1.27 1.27)) (justify right))
     )
@@
       (project "BFMC"
         (path "/a702f17a-d8b6-4710-aaf3-998facd86d1b/c91c3564-35bd-4eac-9426-cc808a6c8173"
-          (reference "R15") (unit 1)
-        )
-      )
+          (reference "R17") (unit 1)
+        )
+      )
